File: 005032.kicad_pcb (KiCad board)
At the start: 2 copper layers, 43 x 26 mm, 47 parts, among them J1 alim+conn, J2 PROG_ESP02, J4 JTAG, SW1 DMR02, SW2 434153017835, SW3 434153017835, U1 ESP32-WROOM-32E, U2 AP63201, U3 AP63357

Commit message: v5 - commit prima di esecuzione modifiche v6
Signed-off-by: Andrea Toninelli <tonazza@yahoo.it>
Parts:
- moved G*** 0.10 mm to (133.7, 92.5)

Commit message: v6 - modificato PCB (TEMP - in attesa revisione meccanica per montaggio su QUANTUM EX 100/150)
Signed-off-by: Andrea Toninelli <tonazza@yahoo.it>
Parts:
- removed C2: 0.1u, Capacitor_SMD:C_0603_1608Metric
- removed the G*** at (105.5, 96.8)
- removed U3: AP63357, aerauliqa-IC:AP6335x
- added D3: STPS0540Z, Diode_SMD:D_SOD-123, F.Cu at (118.6, 97.7)
- added G***: LOGO, aerauliqa-symbols:AQ_logo_pcb_5mm_rame, B.Cu at (125.2, 95.2)
- added R12: 0R33 1%, Resistor_SMD:R_1206_3216Metric_Pad1.42x1.75mm_HandSolder, F.Cu at (106.2, 94.0)
- C3: value 100p -> 220p
- L1: value NRS4018T6R8‎ -> NRS5030T220MMGJ; footprint Inductor_SMD:L_Taiyo-Yuden_NR-40xx -> Inductor_SMD:L_Taiyo-Yuden_NR-50xx
- R1: value 180K 1% -> 11K 1%
- R2, R3: value 57.6K 1% -> 18K 1%
- U2: value AP63201 -> MC34063AD; footprint Package_TO_SOT_SMD:SOT-23-6 -> Package_SO:SOIC-8_3.9x4.9mm_P1.27mm
- moved C1 10.4 mm to (103.4, 90.1)
- moved REF** 7.90 mm to (106.0, 98.0)
- moved C3 6.14 mm to (112.0, 97.3)
- moved R1 4.92 mm to (113.1, 89.8), turned to 180 degrees
- moved R2 4.70 mm to (117.6, 90.1), turned to 180 degrees
- moved TP2 3.86 mm to (102.0, 93.8)
- moved R11 3.84 mm to (103.3, 96.9), turned to 270 degrees
- moved TP3 3.76 mm to (105.2, 93.8), turned to 180 degrees
- moved R10 2.93 mm to (101.6, 96.9)
- moved D1 2.93 mm to (101.6, 93.8)
- moved D2 2.93 mm to (103.3, 93.8)
- moved U2 2.21 mm to (111.2, 93.8), turned to 180 degrees
- moved L1 0.99 mm to (118.1, 93.7)
Connections:
- C3 pad 1: +3V3 -> Net-(C3-Pad1)
- C3 pad 2: Net-(C3-Pad2) -> GND
- R1 pad 1: +3V3 -> Net-(R1-Pad1)
- R1 pad 2: Net-(C3-Pad2) -> GND
- R2 pad 1: Net-(C3-Pad2) -> +3V3
- R2 pad 2: GND -> Net-(R1-Pad1)
- U2 pad 1: Net-(C3-Pad2) -> Net-(R12-Pad2)
- U2 pad 2: +VDC -> /3V3_SW
- U2 pad 3: +VDC -> Net-(C3-Pad1)
- U2 pad 5: /3V3_SW -> Net-(R1-Pad1)
- U2 pad 6: Net-(C2-Pad1) -> +VDC
Routing:
- net +VDC: track 60.1 -> 29.5 mm, vias 6 -> 3
- net Net-(C3-Pad2): track 14.7 -> 0.00 mm, vias 2 -> 0
- net Net-(C2-Pad1): track 12.2 -> 0.00 mm
- net Net-(R1-Pad1): track 0.00 -> 10.6 mm, vias 0 -> 2
- net Net-(R12-Pad2): track 0.00 -> 10.2 mm, vias 0 -> 2
- net GND: track 200.3 -> 190.4 mm, vias 17 -> 16
- net Net-(C3-Pad1): track 0.00 -> 6.27 mm
- net /3V3_SW: track 13.2 -> 7.20 mm
- net +3V3: track 90.9 -> 93.1 mm, vias 4 -> 3
- net /LED_G: track 29.3 -> 27.6 mm, vias 0 -> 2
- net /TXD0: track 33.4 -> 32.0 mm
- net /D1_anode: track 4.26 -> 3.17 mm
- net /D2_anode: track 5.19 -> 4.12 mm
- net /LED_R: track 25.2 -> 26.2 mm
- removed copper zone on F.Cu, net +VDC
- removed copper zone on F.Cu, net /3V3_SW
Other:
- net class Default: clearance 0.15 -> 0.2
- net class power: clearance 0.15 -> 0.2
- rule trace_clearance: 0.15 -> 0.2
- board text added: "005032 v6"
- board text added: "22/02/2022"
- board text added: "Rimossi U3, C2; sostituiti U2, C3, L1, R1, R2, R3; aggiunti R12, D3."
- board text added: "v6"
- board text removed: "005032 v5"
